File: Hardware/triode control board.brd (EAGLE design)
At the start: 99.1 x 83.8 mm, 17 parts, among them J1 JP1

Commit message: switch layout, readme
Parts:
- S1, S2, S3, S4: device SparkFun-mod:SWITCH-SPDT -> SparkFun-Switches:MTS-102-A2
Routing:
- net GND: track 277.5 -> 281.3 mm
- net N$10: track 99.1 -> 100.7 mm
- net N$6: track 56.5 -> 58.0 mm
