File: Hardware/triode control board.sch (EAGLE design)
At the start: 17 parts, among them J1 JP1

Commit message: switch layout, readme
Parts:
- S1, S2, S3, S4: device SparkFun-mod:SWITCH-SPSTMHS122K -> SparkFun-Switches:SWITCH-SPDT
